Commit message: add gravityOff demo

File: urdf/arx5_kdl.urdf (robot description, URDF)
Before this commit: robot urdf6, 7 links, 6 joints
Links:
- link link2: mass 0.601193993090721 -> 0.751193993090721
- link link3: mass 0.912358588332606 -> 0.312358588332606
- link link4: mass 0.288926827428313 -> 0.278926827428313
- link link5: mass 0.312243743001659 -> 0.162243743001659
- link link6: mass 0.284128608326966 -> 0.17425078326966

Commit message: gravity off demo test passed!

File: urdf/arx5_kdl.urdf (robot description, URDF)
Before this commit: robot urdf6, 7 links, 6 joints
Links:
- link link3: mass 0.312358588332606 -> 0.622358588332606
- link link4: mass 0.278926827428313 -> 0.338926827428313
- link link5: mass 0.162243743001659 -> 0.332243743001659
- link link6: mass 0.17425078326966 -> 0.0
